Commit message: Transmision  add to urdf files

File: robot_ejercicio3/urdf/robot_geometry.xacro (robot description, xacro)
@@ -45,6 +45,21 @@
         </link>
     </xacro:macro>
+    <xacro:macro name="wheel_transmission" params="prefix">
+        <!-- Transmisión de las ruedas-->
+        <transmission name="${prefix}_wheel_trans">
+            <type>transmission_interface/SimpleTransmission</type>
+            <joint name="base_${prefix}_wheel_joint">
+                <hardwareInterface>hardware_interface/PositionJointInterface</hardwareInterface>
+            </joint>
+            <actuator name="wheel_motor_${prefix}">
+                <mechanicalReduction>5.0</mechanicalReduction>
+                <hardwareInterface>hardware_interface/PositionJointInterface</hardwareInterface>
+            </actuator>
+        </transmission>
+    </xacro:macro>
     <xacro:wheel_link prefix="left" />
     <xacro:wheel_link prefix="right" />
+    <xacro:wheel_transmission prefix="left" />
+    <xacro:wheel_transmission prefix="right" />
     <link name="lidar_link">
         <visual>
@@ -52,5 +67,5 @@
                 <cylinder radius="${lidar_radius}" length="${lidar_length}" />
             </geometry>
-            <material name="white"/>
+            <material name="white" />
             <origin xyz="0.0 0.0 0.0" rpy="0.0 0.0 0.0" />
         </visual>
