Commit message: listo rviz

File: robot_description/urdf/mobil_base.xacro (robot description, xacro)
@@ -5,6 +5,13 @@
     <xacro:property name="base_height" value="0.0096" />
     <xacro:property name="base_width" value="0.2" />
+    <xacro:property name="base_mass" value="0.5" />
     <xacro:property name="wheel_radius" value="0.02" />
     <xacro:property name="wheel_length" value="0.015" />
+    <xacro:property name="wheel_mass" value="0.1" />
+    <xacro:property name="caster_radius" value="0.03" />
+    <xacro:property name="caster_mass" value="0.005" />
+    <xacro:property name="lidar_radius" value="0.05" />
+    <xacro:property name="lidar_length" value="0.02" />
+    <xacro:property name="lidar_mass" value="0.005" />
     <link name="base_link">
         <visual>
@@ -17,9 +24,10 @@
         </visual>
         <collision>
+            <origin xyz="0 0 0.05" rpy="0 0 0" />
             <geometry>
-                <cylinder radius="${base_width/2}" length="${base_height}" />
+                <cylinder radius="${base_width}" length="${base_height*10}" />
             </geometry>
         </collision>
-        <xacro:cylinder_inertial m="0.5" r="${base_width/2}" l="${base_height}" o_xyz="0 0 0"
+        <xacro:cylinder_inertial m="${base_mass}" r="${base_width/2}" l="${base_height}" o_xyz="0 0 0"
             o_rpy="0 0 0" />
     </link>
@@ -41,9 +49,10 @@
             </visual>
             <collision>
+                <origin xyz="0 0 0" rpy="1.570 0 0" />
                 <geometry>
-                    <cylinder radius="${wheel_radius}" length="${wheel_length}" />
+                    <cylinder radius="${wheel_radius*2}" length="${wheel_length}" />
                 </geometry>
             </collision>
-            <xacro:cylinder_inertial m="0.1" r="${wheel_radius}" l="${wheel_length}" o_xyz="0 0 0"
+            <xacro:cylinder_inertial m="${wheel_mass}" r="${wheel_radius}" l="${wheel_length}" o_xyz="0 0 0"
                 o_rpy="0 0 0" />
         </link>
@@ -62,7 +71,7 @@
             <origin xyz="0 0 0" rpy="0 0 0" />
             <geometry>
-                <sphere radius="0.06" />
+                <sphere radius="${caster_radius}" />
             </geometry>
-            <xacro:sphere_inertial m="0.01" r="0.06" o_xyz="0 0 0" o_rpy="0 0 0" />
+            <xacro:sphere_inertial m="${caster_mass}" r="${caster_radius*2}" o_xyz="0 0 0" o_rpy="0 0 0" />
         </collision>
     </link>
@@ -79,7 +88,7 @@
             <origin xyz="0 0 0" rpy="0 0 0" />
             <geometry>
-                <cylinder radius="0.05" length="0.02" />
+                <cylinder radius="${lidar_radius}" length="${lidar_length}" />
             </geometry>
-            <xacro:cylinder_inertial m="0.05" r="0.05" l="0.02" o_xyz="0 0 0" o_rpy="0 0 0" />
+            <xacro:cylinder_inertial m="${lidar_mass}" r="${lidar_radius}" l="${lidar_length}" o_xyz="0 0 0" o_rpy="0 0 0" />
         </collision>
     </link>

Commit message: Robot moviendose en gazebo

File: robot_description/urdf/mobil_base.xacro (robot description, xacro)
@@ -20,5 +20,5 @@
                     scale="0.001 0.001 0.001" />
             </geometry>
-            <origin xyz="0 0 0" rpy="0 0 0" />
+            <origin xyz="0 0 ${wheel_radius/2}" rpy="0 0 0" />
             <material name="white" />
         </visual>
@@ -90,6 +90,6 @@
                 <cylinder radius="${lidar_radius}" length="${lidar_length}" />
             </geometry>
-            <xacro:cylinder_inertial m="${lidar_mass}" r="${lidar_radius}" l="${lidar_length}" o_xyz="0 0 0" o_rpy="0 0 0" />
         </collision>
+          <xacro:cylinder_inertial m="${lidar_mass}" r="${lidar_radius}" l="${lidar_length}" o_xyz="0 0 0" o_rpy="0 0 0" />
     </link>
     <joint name="right_wheel_joint" type="continuous">

File: robot_description/urdf/robot_final.urdf.xacro (robot description, xacro)
@@ -3,3 +3,4 @@
     <xacro:include filename="$(find robot_description)/urdf/common_properties.xacro"/>
     <xacro:include filename="$(find robot_description)/urdf/mobil_base.xacro"/>
+    <xacro:include filename="$(find robot_description)/urdf/mobil_base_gazebo.xacro"/>
 </robot>
